Commit message: Updated vessel model

File: catkin_ws/src/simulator_prototype/config/models/Odin.urdf (robot description, URDF)
Before this commit: robot hil_sim, 1 links, 0 joints
Links:
- link hil_sim: geometry visual mesh filename=file:///home/d943/Dropbox/Master2/OdinDecimated.stl scale=0.001 0.001 0.001
