Commit message: Updated nonlinear surge damping

File: catkin_ws/src/simulator_prototype/config/models/Jolner.urdf (robot description, URDF)
Before this commit: robot hil_sim, 1 links, 0 joints
Links:
- link hil_sim: geometry visual mesh filename=file:///home/Jolner.stl scale=0.01 0.01 0.01

File: catkin_ws/src/simulator_prototype/config/models/Odin.urdf (robot description, URDF)
Before this commit: robot hil_sim, 1 links, 0 joints
Links:
- link hil_sim: geometry visual mesh filename=file:///home/OdinDecimated.stl scale=0.001 0.001 0.001
